Commit message: new dense point cloud

File: datasets/arm/UR5/ur5e.urdf (robot description, URDF)
Before this commit: robot ur5e_robot, 11 links, 10 joints
Links:
- link base_link_inertia: geometry collision mesh filename=meshes/collision/base.stl; visual mesh filename=meshes/visual/base.dae
- link forearm_link: geometry collision mesh filename=meshes/collision/forearm.stl; visual mesh filename=meshes/visual/forearm.dae
- link shoulder_link: geometry collision mesh filename=meshes/collision/shoulder.stl; visual mesh filename=meshes/visual/shoulder.dae
- link upper_arm_link: geometry collision mesh filename=meshes/collision/upperarm.stl; visual mesh filename=meshes/visual/upperarm.dae
- link wrist_1_link: geometry collision mesh filename=meshes/collision/wrist_1.stl; visual mesh filename=meshes/visual/wrist1.dae
- link wrist_2_link: geometry collision mesh filename=meshes/collision/wrist_2.stl; visual mesh filename=meshes/visual/wrist2.dae
- link wrist_3_link: geometry collision mesh filename=meshes/collision/wrist_3.stl; visual mesh filename=meshes/visual/wrist3.dae
